Commit message: Finished sensors

File: body.urdf (robot description, URDF)
Before this commit: robot robot, 3 links, 2 joints
Links:
- removed link Backleg
- removed link Frontleg
- added link BackLeg, mass 1; collision box size=1 1 1; visual box size=1 1 1
- added link FrontLeg, mass 1; collision box size=1 1 1; visual box size=1 1 1
Joints:
- removed joint Torso_Backleg
- removed joint Torso_Frontleg
- added joint Torso_BackLeg: type revolute, parent Torso, child BackLeg, origin xyz=2 0 1 rpy=0 0 0, axis 0 1 0, limit lower=-3.14159 upper=3.14159 effort=0.0 velocity=0.0
- added joint Torso_FrontLeg: type revolute, parent Torso, child FrontLeg, origin xyz=1 0 1 rpy=0 0 0, axis 0 1 0, limit lower=-3.14159 upper=3.14159 effort=0.0 velocity=0.0

Commit message: finished parallelhc 2

File: body.urdf (robot description, URDF)
Before this commit: robot robot, 3 links, 2 joints
Joints:
- joint Torso_BackLeg: origin xyz=2 0 1 rpy=0 0 0 -> xyz=1 0 1 rpy=0 0 0
- joint Torso_FrontLeg: origin xyz=1 0 1 rpy=0 0 0 -> xyz=2 0 1 rpy=0 0 0

Commit message: finished quadruped

File: body.urdf (robot description, URDF)
Before this commit: robot robot, 3 links, 2 joints
Links:
- added link BackLowerLeg, mass 1; collision box size=0.2 0.2 1; visual box size=0.2 0.2 1
- added link FrontLowerLeg, mass 1; collision box size=0.2 0.2 1; visual box size=0.2 0.2 1
- added link LeftLeg, mass 1; collision box size=1 0.2 0.2; visual box size=1 0.2 0.2
- added link LeftLowerLeg, mass 1; collision box size=0.2 0.2 1; visual box size=0.2 0.2 1
- added link RightLeg, mass 1; collision box size=1 0.2 0.2; visual box size=1 0.2 0.2
- added link RightLowerLeg, mass 1; collision box size=0.2 0.2 1; visual box size=0.2 0.2 1
- link BackLeg: geometry collision box size=0.2 -1 0.2; visual box size=0.2 -1 0.2
- link FrontLeg: geometry collision box size=0.2 1 0.2; visual box size=0.2 1 0.2
Joints:
- added joint BackLeg_BackLowerLeg: type revolute, parent BackLeg, child BackLowerLeg, origin xyz=0 -1 0 rpy=0 0 0, axis 1 0 0, limit lower=-3.14159 upper=3.14159 effort=0.0 velocity=0.0
- added joint FrontLeg_FrontLowerLeg: type revolute, parent FrontLeg, child FrontLowerLeg, origin xyz=0 1 0 rpy=0 0 0, axis 1 0 0, limit lower=-3.14159 upper=3.14159 effort=0.0 velocity=0.0
- added joint LeftLeg_LeftLowerLeg: type revolute, parent LeftLeg, child LeftLowerLeg, origin xyz=-1 0 0 rpy=0 0 0, axis 0 1 0, limit lower=-3.14159 upper=3.14159 effort=0.0 velocity=0.0
- added joint RightLeg_RightLowerLeg: type revolute, parent RightLeg, child RightLowerLeg, origin xyz=1 0 0 rpy=0 0 0, axis 0 1 0, limit lower=-3.14159 upper=3.14159 effort=0.0 velocity=0.0
- added joint Torso_LeftLeg: type revolute, parent Torso, child LeftLeg, origin xyz=-0.5 0 1 rpy=0 0 0, axis 0 1 0, limit lower=-3.14159 upper=3.14159 effort=0.0 velocity=0.0
- added joint Torso_RightLeg: type revolute, parent Torso, child RightLeg, origin xyz=0.5 0 1 rpy=0 0 0, axis 0 1 0, limit lower=-3.14159 upper=3.14159 effort=0.0 velocity=0.0
- joint Torso_BackLeg: axis 0 1 0 -> 1 0 0; origin xyz=1 0 1 rpy=0 0 0 -> xyz=0 -0.5 1 rpy=0 0 0
- joint Torso_FrontLeg: axis 0 1 0 -> 1 0 0; origin xyz=2 0 1 rpy=0 0 0 -> xyz=0 0.5 1 rpy=0 0 0

Commit message: final project

File: body.urdf (robot description, URDF)
Before this commit: robot robot, 9 links, 8 joints
Links:
- removed link BackLeg
- removed link BackLowerLeg
- removed link FrontLowerLeg
- removed link LeftLeg
- removed link LeftLowerLeg
- removed link RightLowerLeg
- added link Front2Leg, mass 1; collision box size=0.05 1 0.05; visual box size=0.05 1 0.05
- added link Front3Leg, mass 1; collision box size=0.05 1 0.05; visual box size=0.05 1 0.05
- added link Front4Leg, mass 1; collision box size=0.05 0.05 0.1; visual box size=0.05 0.05 0.1
- link FrontLeg: geometry collision box size=0.05 1 0.05; visual box size=0.05 1 0.05
- link RightLeg: geometry collision box size=0.05 1 0.05; visual box size=0.05 1 0.05
- link Torso: geometry collision box size=1 0.5 0.05; visual box size=1 0.5 0.05
Joints:
- removed joint BackLeg_BackLowerLeg
- removed joint FrontLeg_FrontLowerLeg
- removed joint LeftLeg_LeftLowerLeg
- removed joint RightLeg_RightLowerLeg
- removed joint Torso_BackLeg
- removed joint Torso_LeftLeg
- added joint Torso_Front2Leg: type revolute, parent Torso, child Front2Leg, origin xyz=-0.4 0.1 1.05 rpy=0 0 0, axis 1 0 0, limit lower=-3.14159 upper=3.14159 effort=0.0 velocity=0.0
- added joint Torso_Front3Leg: type revolute, parent Torso, child Front3Leg, origin xyz=0.4 0.1 1.05 rpy=0 0 0, axis 1 0 0, limit lower=-3.14159 upper=3.14159 effort=0.0 velocity=0.0
- added joint Torso_Front4Leg: type revolute, parent Torso, child Front4Leg, origin xyz=0.5 0.06 0.02 rpy=0 0 0, axis 0 1 0, limit lower=-3.14159 upper=3.14159 effort=0.0 velocity=0.0
- joint Torso_FrontLeg: origin xyz=0 0.5 1 rpy=0 0 0 -> xyz=-0.1 0.1 1.05 rpy=0 0 0
- joint Torso_RightLeg: axis 0 1 0 -> 1 0 0; origin xyz=0.5 0 1 rpy=0 0 0 -> xyz=0.1 0.1 1.05 rpy=0 0 0

Commit message: random snake

File: body.urdf (robot description, URDF)
Before this commit: robot robot, 6 links, 5 joints
Links:
- removed link Front2Leg
- removed link Front3Leg
- removed link Front4Leg
- removed link FrontLeg
- removed link RightLeg
- added link bladder, mass 1; collision box size=0.28305855185581497 0.7042561274183264 0.15372420304624268; visual box size=0.28305855185581497 0.7042561274183264 0.15372420304624268
- added link finger, mass 1; collision box size=0.7319327913142831 0.8644973587842858 0.9985708215268283; visual box size=0.7319327913142831 0.8644973587842858 0.9985708215268283
- added link heart, mass 1; collision box size=0.8817672399556126 0.6900020409402926 0.7921315783068796; visual box size=0.8817672399556126 0.6900020409402926 0.7921315783068796
- added link intestine, mass 1; collision box size=0.0545329682920046 0.9718885179653312 0.9687772159828055; visual box size=0.0545329682920046 0.9718885179653312 0.9687772159828055
- added link kidney, mass 1; collision box size=0.055469185660437126 0.855246027502417 0.27780710591550173; visual box size=0.055469185660437126 0.855246027502417 0.27780710591550173
- added link leg, mass 1; collision box size=0.16680816586459035 0.5191346406634993 0.39203835599980796; visual box size=0.16680816586459035 0.5191346406634993 0.39203835599980796
- added link lungs, mass 1; collision box size=0.8948685531746331 0.34111743394323346 0.2095707914171272; visual box size=0.8948685531746331 0.34111743394323346 0.2095707914171272
- added link stomach, mass 1; collision box size=0.7040876225404046 0.163236120055133 0.4487204597128963; visual box size=0.7040876225404046 0.163236120055133 0.4487204597128963
- link Torso: geometry collision box size=1.3175645076584712 1 1; visual box size=1.3175645076584712 1 1
Joints:
- removed joint Torso_Front2Leg
- removed joint Torso_Front3Leg
- removed joint Torso_Front4Leg
- removed joint Torso_FrontLeg
- removed joint Torso_RightLeg
- added joint Torso_lungs: type revolute, parent Torso, child lungs, origin xyz=-3.3412177461707646 0 3 rpy=0 0 0, axis 0 1 0, limit lower=-3.14159 upper=3.14159 effort=0.0 velocity=0.0
- added joint bladder_kidney: type revolute, parent bladder, child kidney, origin xyz=0.28305855185581497 0 0 rpy=0 0 0, axis 0 1 0, limit lower=-3.14159 upper=3.14159 effort=0.0 velocity=0.0
- added joint finger_leg: type revolute, parent finger, child leg, origin xyz=0.7319327913142831 0 0 rpy=0 0 0, axis 0 1 0, limit lower=-3.14159 upper=3.14159 effort=0.0 velocity=0.0
- added joint heart_finger: type revolute, parent heart, child finger, origin xyz=0.8817672399556126 0 0 rpy=0 0 0, axis 0 1 0, limit lower=-3.14159 upper=3.14159 effort=0.0 velocity=0.0
- added joint intestine_heart: type revolute, parent intestine, child heart, origin xyz=0.0545329682920046 0 0 rpy=0 0 0, axis 0 1 0, limit lower=-3.14159 upper=3.14159 effort=0.0 velocity=0.0
- added joint kidney_stomach: type revolute, parent kidney, child stomach, origin xyz=0.055469185660437126 0 0 rpy=0 0 0, axis 0 1 0, limit lower=-3.14159 upper=3.14159 effort=0.0 velocity=0.0
- added joint lungs_bladder: type revolute, parent lungs, child bladder, origin xyz=0.8948685531746331 0 0 rpy=0 0 0, axis 0 1 0, limit lower=-3.14159 upper=3.14159 effort=0.0 velocity=0.0
- added joint stomach_intestine: type revolute, parent stomach, child intestine, origin xyz=0.7040876225404046 0 0 rpy=0 0 0, axis 0 1 0, limit lower=-3.14159 upper=3.14159 effort=0.0 velocity=0.0
